Commit message: include new world file and updated launch and urdf

File: urdf/jackal_ouster.urdf.xacro (robot description, xacro)
@@ -1,6 +1,6 @@
 <?xml version="1.0"?>
 <robot name="jackal_ouster" xmlns:xacro="https://ros.org/wiki/xacro">
+  <xacro:include filename="$(find jackal_description)/urdf/jackal.urdf.xacro" />
   <xacro:include filename="$(find jackal_gazebo_simulations/urdf/jackal_ouster.gazebo.xacro"/>
-  <xacro:property name="PI" value="3.1415926535897931"/>
   <xacro:property name="ouster_px" value="0.0"/>
   <xacro:property name="ouster_py" value="0.0"/>

Commit message: update launch and urdf and add gazebo.xacro file

File: urdf/jackal_ouster.urdf.xacro (robot description, xacro)
@@ -1,13 +1,234 @@
 <?xml version="1.0"?>
 <robot name="jackal_ouster" xmlns:xacro="https://ros.org/wiki/xacro">
-  <xacro:include filename="$(find jackal_description)/urdf/jackal.urdf.xacro" />
-  <xacro:include filename="$(find jackal_gazebo_simulations/urdf/jackal_ouster.gazebo.xacro"/>
+  <xacro:property name="PI" value="3.1415926535897931"/>
   <xacro:property name="ouster_px" value="0.0"/>
   <xacro:property name="ouster_py" value="0.0"/>
   <xacro:property name="ouster_pz" value="0.0"/>
+  <xacro:property name="wheelbase" value="0.262" />
+  <xacro:property name="track" value="0.37559" />
+  <xacro:property name="wheel_vertical_offset" value="0.0345" />
+  <xacro:property name="footprint_vertical_offset" value="-0.0655" />
+  <xacro:property name="wheel_radius" value="0.098" />
+  <xacro:property name="wheel_width" value="0.040" />
+  <xacro:property name="chassis_length" value="0.420" />
+  <xacro:property name="chassis_width" value="0.310" />
+  <xacro:property name="chassis_height" value="0.184" />
+  <xacro:property name="dummy_inertia" value="1e-09"/>
+  <xacro:property name="mount_spacing" value="0.120" />
+  <material name="dark_grey"><color rgba="0.2 0.2 0.2 1.0" /></material>
+  <material name="light_grey"><color rgba="0.4 0.4 0.4 1.0" /></material>
+  <material name="yellow"><color rgba="0.8 0.8 0.0 1.0" /></material>
+  <material name="black"><color rgba="0.15 0.15 0.15 1.0" /></material>
+  <xacro:macro name="wheel" params="prefix *joint_pose">
+    <link name="${prefix}_wheel_link">
+      <visual>
+        <origin xyz="0 0 0" rpy="${PI/2} 0 0"/>
+        <geometry>
+          <mesh filename="package://jackal_description/meshes/jackal-wheel.stl"/>
+        </geometry>
+        <material name="black" />
+      </visual>
+      <collision>
+        <origin xyz="0 0 0" rpy="${PI/2} 0 0"/>
+        <geometry>
+          <cylinder radius="${wheel_radius}" length="${wheel_width}"/>
+        </geometry>
+      </collision>
+      <inertial>
+        <origin xyz="0 0 0" rpy="0 0 0"/>
+        <mass value="0.477"/>
+        <inertia
+          ixx="0.0013" ixy="0" ixz="0"
+          iyy="0.0024" iyz="0"
+          izz="0.0013"/>
+      </inertial>
+    </link>
+    <gazebo reference="${prefix}_wheel_link">
+      <material>Gazebo/DarkGrey</material>
+      <selfCollide>false</selfCollide>
+      <mu1 value="0.5"/>
+      <mu2 value="0.5"/>
+      <kp value="10000000.0" />
+      <kd value="1" />
+      <fdir1 value="1 0 0"/>
+    </gazebo>
+    <joint name="${prefix}_wheel" type="continuous">
+      <parent link="chassis_link"/>
+      <child link="${prefix}_wheel_link" />
+      <xacro:insert_block name="joint_pose" />
+      <axis xyz="0 1 0" />
+    </joint>
+    <!-- In reality, Jackal has only two motors, one per side. However, it's more
+         straightforward for Gazebo to simulate as if there's an actuator per wheel. -->
+    <transmission name="${prefix}_wheel_trans">
+      <type>transmission_interface/SimpleTransmission</type>
+      <joint name="${prefix}_wheel">
+        <hardwareInterface>hardware_interface/VelocityJointInterface</hardwareInterface>
+      </joint>
+      <actuator name="${prefix}_actuator">
+        <mechanicalReduction>1</mechanicalReduction>
+      </actuator>
+    </transmission>
+  </xacro:macro>
+  <xacro:wheel prefix="front_left">
+    <origin xyz="${wheelbase/2} ${track/2} ${wheel_vertical_offset}" rpy="0 0 0" />
+  </xacro:wheel>
+  <xacro:wheel prefix="front_right">
+    <origin xyz="${wheelbase/2} ${-track/2} ${wheel_vertical_offset}" rpy="0 0 0" />
+  </xacro:wheel>
+  <xacro:wheel prefix="rear_left">
+    <origin xyz="${-wheelbase/2} ${track/2} ${wheel_vertical_offset}" rpy="0 0 0" />
+  </xacro:wheel>
+  <xacro:wheel prefix="rear_right">
+    <origin xyz="${-wheelbase/2} ${-track/2} ${wheel_vertical_offset}" rpy="0 0 0" />
+  </xacro:wheel>
   <link name="base_link"></link>
   <joint name="base_link_joint" type="fixed">
     <origin xyz="0 0 0" rpy="0 0 0" />
-    <parent link="base_link" />
+    <parent link="base_link"/>
     <child link="chassis_link" />
   </joint>
+  <link name="chassis_link">
+    <visual>
+      <origin xyz="0 0 ${footprint_vertical_offset}" rpy="${PI/2} 0 ${PI/2}"/>
+      <geometry>
+        <mesh filename="package://jackal_description/meshes/jackal-base.stl"/>
+      </geometry>
+      <material name="dark_grey" />
+    </visual>
+    <collision>
+      <origin xyz="0 0 ${chassis_height/2}"/>
+      <geometry>
+        <box size="${chassis_length} ${chassis_width} ${chassis_height}"/>
+      </geometry>
+    </collision>
+    <inertial>
+      <!-- Center of mass -->
+      <origin xyz="0.012  0.002 0.067" rpy="0 0 0"/>
+      <mass value="16.523"/>
+      <!-- Moments of inertia: ( chassis without wheels ) -->
+      <inertia
+        ixx="0.3136" ixy="-0.0008" ixz="0.0164"
+        iyy="0.3922" iyz="-0.0009"
+        izz="0.4485"/>
+      </inertial>
+  </link>
+  <xacro:unless value="$(optenv JACKAL_FRONT_ACCESSORY_FENDER 0)">
+    <link name="front_fender_link">
+      <visual>
+        <geometry>
+          <mesh filename="package://jackal_description/meshes/jackal-fender.stl"/>
+        </geometry>
+        <material name="yellow" />
+      </visual>
+    </link>
+  </xacro:unless>
+  <xacro:if value="$(optenv JACKAL_FRONT_ACCESSORY_FENDER 0)">
+    <link name="front_fender_link">
+      <visual>
+        <geometry>
+          <mesh filename="package://jackal_description/meshes/accessory_fender.stl"/>
+        </geometry>
+        <material name="yellow" />
+      </visual>
+    </link>
+    <link name="front_fender_accessory_link"/>
+    <joint name="front_fender_accessory_joint" type="fixed">
+      <origin xyz="0.25629 0 0.07455" rpy="${PI} 0 0" />
+      <parent link="front_fender_link" />
+      <child link="front_fender_accessory_link" />
+    </joint>
+  </xacro:if>
+  <joint name="front_fender_joint" type="fixed">
+    <origin xyz="0 0 0" rpy="0 0 0"/>
+    <parent link="chassis_link" />
+    <child link="front_fender_link" />
+  </joint>
+  <xacro:unless value="$(optenv JACKAL_REAR_ACCESSORY_FENDER 0)">
+    <link name="rear_fender_link">
+      <visual>
+        <geometry>
+          <mesh filename="package://jackal_description/meshes/jackal-fender.stl"/>
+        </geometry>
+        <material name="yellow" />
+      </visual>
+    </link>
+  </xacro:unless>
+  <xacro:if value="$(optenv JACKAL_REAR_ACCESSORY_FENDER 0)">
+    <link name="rear_fender_link">
+      <visual>
+        <geometry>
+          <mesh filename="package://jackal_description/meshes/accessory_fender.stl"/>
+        </geometry>
+        <material name="yellow" />
+      </visual>
+    </link>
+    <link name="rear_fender_accessory_link"/>
+    <joint name="rear_fender_accessory_joint" type="fixed">
+      <origin xyz="0.25629 0 0.07455" rpy="${PI} 0 0" />
+      <parent link="rear_fender_link" />
+      <child link="rear_fender_accessory_link" />
+    </joint>
+  </xacro:if>
+  <joint name="rear_fender_joint" type="fixed">
+    <origin xyz="0 0 0" rpy="0 0 ${PI}"/>
+    <parent link="chassis_link" />
+    <child link="rear_fender_link" />
+  </joint>
+  <!-- TODO: Make this internal_imu_link or something, and use a mixed-in xacro
+       to supply the joint between it and imu_link. This is important so that imu_link
+       always points to the "active" IMU. When an upgrade IMU is connected, the
+       internal_imu_link should remain, but imu_link should point to the upgrade one. -->
+  <link name="imu_link">
+    <inertial>
+      <mass value="0.001"/>
+      <origin xyz="0 0 0" rpy="0 0 0"/>
+      <inertia ixx="${dummy_inertia}" ixy="0.0" ixz="0.0" iyy="${dummy_inertia}" iyz="0.0" izz="${dummy_inertia}"/>
+    </inertial>
+  </link>
+  <joint name="imu_joint" type="fixed">
+    <parent link="chassis_link" />
+    <child link="imu_link" />
+  </joint>
+  <!-- TODO: Same note as applies to imu_link -->
+  <link name="navsat_link">
+    <visual>
+      <geometry>
+        <cylinder radius="0.026" length="0.016" />
+      </geometry>
+      <origin xyz="0 0 0.008" />
+      <material name="black" />
+    </visual>
+  </link>
+  <joint name="navsat_joint" type="fixed">
+    <parent link="chassis_link" />
+    <child link="navsat_link" />
+    <origin xyz="-0.180 0.126 0.1815" />
+  </joint>
+  <link name="mid_mount"></link>
+  <joint name="mid_mount_joint" type="fixed">
+    <parent link="chassis_link" />
+    <child link="mid_mount" />
+    <origin xyz="0 0 ${chassis_height}" />
+  </joint>
+  <link name="rear_mount"></link>
+  <joint name="rear_mount_joint" type="fixed">
+    <parent link="mid_mount" />
+    <child link="rear_mount" />
+    <origin xyz="${-mount_spacing} 0 0" />
+  </joint>
+  <link name="front_mount"></link>
+  <joint name="front_mount_joint" type="fixed">
+    <parent link="mid_mount" />
+    <child link="front_mount" />
+    <origin xyz="${mount_spacing} 0 0" />
+  </joint>
+  <!-- Bring in simulation data for Gazebo. -->
+  <xacro:include filename="$(find jackal_gazebo_simulations)/urdf/jackal_ouster.gazebo.xacro"/>
+  <!-- Optional standard accessories, including their simulation data. The rendering
+       of these into the final description is controlled by optenv variables, which
+       default each one to off.-->
+  <xacro:include filename="$(find jackal_description)/urdf/accessories.urdf.xacro" />
+  <!-- Optional custom includes. -->
+  <!--xacro:include filename="$(optenv JACKAL_URDF_EXTRAS empty.urdf)" /-->
+</robot>

Commit message: added OS1 in urdf

File: urdf/jackal_ouster.urdf.xacro (robot description, xacro)
@@ -224,4 +224,17 @@
     <origin xyz="${mount_spacing} 0 0" />
   </joint>
+  <!-- This field for Ouster OS1-32-->
+  <xacro:property name="lidar_parent_link" value="front_mount"/>
+  <xacro:include filename="$(find ouster_os1_64)/urdf/os1_64.urdf.xacro"/>
+  <xacro:os1_64 parent="${lidar_parent_link}"
+		name="ouster"
+		prefix="/os1_cloud_node"
+		hz="10"
+		samples="2048"
+		v_samples="64"
+		reduced="false"
+		gpu="true">
+    <origin xyz="${ouster_px} ${ouster_py} ${ouster_pz}" rpy="0 0 0" />
+  </xacro:os1_64>
   <!-- Bring in simulation data for Gazebo. -->
   <xacro:include filename="$(find jackal_gazebo_simulations)/urdf/jackal_ouster.gazebo.xacro"/>
@@ -229,5 +242,5 @@
        of these into the final description is controlled by optenv variables, which
        default each one to off.-->
-  <xacro:include filename="$(find jackal_description)/urdf/accessories.urdf.xacro" />
+  <!-- xacro:include filename="$(find jackal_description)/urdf/accessories.urdf.xacro" /-->
   <!-- Optional custom includes. -->
   <!--xacro:include filename="$(optenv JACKAL_URDF_EXTRAS empty.urdf)" /-->

Commit message: update urdf and test in Gazebo

File: urdf/jackal_ouster.urdf.xacro (robot description, xacro)
@@ -4,5 +4,5 @@
   <xacro:property name="ouster_px" value="0.0"/>
   <xacro:property name="ouster_py" value="0.0"/>
-  <xacro:property name="ouster_pz" value="0.0"/>
+  <xacro:property name="ouster_pz" value="0.25"/>
   <xacro:property name="wheelbase" value="0.262" />
   <xacro:property name="track" value="0.37559" />
@@ -225,13 +225,18 @@
   </joint>
   <!-- This field for Ouster OS1-32-->
-  <xacro:property name="lidar_parent_link" value="front_mount"/>
+  <xacro:property name="lidar_parent_link" value="mid_mount"/>
   <xacro:include filename="$(find ouster_os1_64)/urdf/os1_64.urdf.xacro"/>
   <xacro:os1_64 parent="${lidar_parent_link}"
 		name="ouster"
 		prefix="/os1_cloud_node"
+    min_angle_v="-22.5"
+    max_angle_v="22.5"
+    min_range="0.15"
+    max_range="100"
 		hz="10"
-		samples="2048"
+		samples="1024"
 		v_samples="64"
-		reduced="false"
+    noise="0.001"
+		reduced="true"
 		gpu="true">
     <origin xyz="${ouster_px} ${ouster_py} ${ouster_pz}" rpy="0 0 0" />

Commit message: update urdf and launch file, test lio-sam

File: urdf/jackal_ouster.urdf.xacro (robot description, xacro)
@@ -4,5 +4,5 @@
   <xacro:property name="ouster_px" value="0.0"/>
   <xacro:property name="ouster_py" value="0.0"/>
-  <xacro:property name="ouster_pz" value="0.25"/>
+  <xacro:property name="ouster_pz" value="0.0"/>
   <xacro:property name="wheelbase" value="0.262" />
   <xacro:property name="track" value="0.37559" />
@@ -236,5 +236,5 @@
 		hz="10"
 		samples="1024"
-		v_samples="64"
+		v_samples="32"
     noise="0.001"
 		reduced="true"
