Commit message: update urdf and tune param

File: urdf/jackal_ouster.gazebo.xacro (robot description, xacro)
@@ -13,9 +13,9 @@
       <topicName>imu/data</topicName>
       <accelDrift>0.005 0.005 0.005</accelDrift>
-      <accelGaussianNoise>0.005 0.005 0.005</accelGaussianNoise>
+      <accelGaussianNoise>0.000 0.000 0.000</accelGaussianNoise>
       <rateDrift>0.005 0.005 0.005 </rateDrift>
-      <rateGaussianNoise>0.005 0.005 0.005 </rateGaussianNoise>
-      <headingDrift>0.005</headingDrift>
-      <headingGaussianNoise>0.005</headingGaussianNoise>
+      <rateGaussianNoise>0.000 0.000 0.000 </rateGaussianNoise>
+      <headingDrift>0.000</headingDrift>
+      <headingGaussianNoise>0.000</headingGaussianNoise>
     </plugin>
   </gazebo>

File: urdf/jackal_ouster.urdf.xacro (robot description, xacro)
@@ -4,5 +4,5 @@
   <xacro:property name="ouster_px" value="0.0"/>
   <xacro:property name="ouster_py" value="0.0"/>
-  <xacro:property name="ouster_pz" value="0.0"/>
+  <xacro:property name="ouster_pz" value="0.4"/>
   <xacro:property name="wheelbase" value="0.262" />
   <xacro:property name="track" value="0.37559" />
@@ -225,5 +225,5 @@
   </joint>
   <!-- This field for Ouster OS1-32-->
-  <xacro:property name="lidar_parent_link" value="mid_mount"/>
+  <xacro:property name="lidar_parent_link" value="chassis_link"/>
   <xacro:include filename="$(find ouster_os1_64)/urdf/os1_64.urdf.xacro"/>
   <xacro:os1_64 parent="${lidar_parent_link}"
@@ -235,5 +235,5 @@
     max_range="100"
 		hz="10"
-		samples="1024"
+		samples="512"
 		v_samples="32"
     noise="0.001"
